Commit message: FIX Upload vehicle with inertial frame world_ned
Signed-off-by: Musa Morena Marcusso Manhaes <Musa.Marcusso@de.bosch.com>

File: lauv_description/robots/default.xacro (robot description, xacro)
@@ -3,9 +3,12 @@
   <xacro:arg name="debug" default="0"/>
   <xacro:arg name="namespace" default="lauv"/>
+  <xacro:arg name="inertial_reference_frame" default="world"/>
   <!-- Include the ROV macro file -->
   <xacro:include filename="$(find lauv_description)/urdf/base.xacro"/>
   <xacro:include filename="$(find lauv_description)/urdf/gazebo.xacro"/>
   <!-- Create the lauv -->
-  <xacro:lauv_base namespace="$(arg namespace)">
+  <xacro:lauv_base
+    namespace="$(arg namespace)"
+    inertial_reference_frame="$(arg inertial_reference_frame)">
     <!-- The underwater object plugin is given as an input block parameter to
      allow the addition of external models of manipulator units -->

File: lauv_description/urdf/base.xacro (robot description, xacro)
@@ -29,5 +29,5 @@
   <xacro:property name="collision_mesh_file" value="file://$(find lauv_description)/meshes/body.stl"/>
   <!-- Vehicle macro -->
-  <xacro:macro name="lauv_base" params="namespace *gazebo">
+  <xacro:macro name="lauv_base" params="namespace *gazebo inertial_reference_frame">
       <!-- Rigid body description of the base link -->
       <link name="${namespace}/base_link">

File: lauv_description/urdf/sensors.xacro (robot description, xacro)
@@ -10,5 +10,8 @@
   <xacro:default_gps namespace="${namespace}" parent_link="${namespace}/base_link" />
   <!-- Mount a Pose 3D sensor. -->
-  <xacro:default_pose_3d namespace="${namespace}" parent_link="${namespace}/base_link" />
+  <xacro:default_pose_3d_macro
+    namespace="${namespace}"
+    parent_link="${namespace}/base_link"
+    inertial_reference_frame="${inertial_reference_frame}" />
   <!-- Forward-looking sonar sensor -->
   <!-- <xacro:forward_multibeam_p900 namespace="${namespace}" parent_link="${namespace}/base_link">
